Commit message: 打通 Piper mock 控制链路
- 新增 unistackbot_hardware_mock 包,实现 MockPiperHardware 插件(速度限幅积分)
- piper_ros2_control.xacro 切换插件为 MockPiperHardware,清理 ros2_control 块内的 mimic joint
- unistackbot_bringup 加 piper_controllers.yaml 与 piper_control.launch.py,拉起 robot_state_publisher + ros2_control_node

Co-Authored-By: Claude Opus 4.7 <noreply@anthropic.com>

File: unistackbot_description/arms/piper/urdf/piper_ros2_control.xacro (robot description, xacro)
@@ -4,5 +4,5 @@
         <ros2_control name="piper_system" type="system">
             <hardware>
-                <plugin>unistackbot_hardware/PiperSystem</plugin>
+                <plugin>unistackbot_hardware_mock/MockPiperHardware</plugin>
                 <param name="device">/dev/piper_arm</param>
                 <param name="baudrate">2000000</param>
@@ -65,12 +65,4 @@
                     <param name="max">0.1</param>
                 </joint>
-                <joint name="gripper_joint1">
-                    <param name="mimic">gripper</param>
-                    <param name="multiplier">0.5</param>
-                </joint>
-                <joint name="gripper_joint2">
-                    <param name="mimic">gripper</param>
-                    <param name="multiplier">-0.5</param>
-                </joint>
             </xacro:if>
         </ros2_control>
