Commit message: 仿真三包归组进unistackbot_sim_control/容器目录(core/gazebo/mujoco, 包名不变); gz 0.7.21适配:piper手指ign分支改state-only修激活, gripper不响应遗留入档

File: unistackbot_description/arms/piper/urdf/piper_ros2_control.xacro (robot description, xacro)
@@ -93,8 +93,12 @@
                 </joint>
                 <!-- 两个 mimic 手指关节, 按链分流:
-                     mujoco: passive (MJCF 侧 equality 耦合跟随 gripper, 见 mujoco/README.md),
-                             无 command_interface → JointStream 解析后只管 7 个主关节
-                     其余 (mock/gz): 按 gazebo_ros2_control 要求补 mimic/multiplier 参数受控跟随 -->
-                <xacro:if value="${use_gazebo == 'mujoco'}">
+                     mujoco/ign: passive —— 无 command_interface, 跟随由仿真侧原生 mimic 语义承担
+                       (mujoco: MJCF equality, 见 mujoco/README.md; gz 0.7.21+: URDF <mimic> 标签,
+                       插件原生处理)。JointStream 解析后只管 7 个主关节。
+                       2026-09-21 实测: gz_ros2_control 升级 0.7.21 后 (mujoco 安装的 apt 连带),
+                       带 mimic 参数声明手指会被导出为 <joint>_mimic 接口名 → JS 声明 9 关节对不上
+                       "Not acceptable command interfaces combination"。
+                     mock/Classic: 按 gazebo_ros2_control 要求补 mimic/multiplier 参数受控跟随 -->
+                <xacro:if value="${use_gazebo in ['mujoco', 'ign']}">
                     <joint name="gripper_joint1">
                         <state_interface name="position"/>
@@ -106,5 +110,5 @@
                     </joint>
                 </xacro:if>
-                <xacro:unless value="${use_gazebo == 'mujoco'}">
+                <xacro:unless value="${use_gazebo in ['mujoco', 'ign']}">
                     <joint name="gripper_joint1">
                         <command_interface name="position"/>

Commit message: gz链关节冻结修复: ign分支joint2/joint3/gripper加initial_value离限位线(上游gz_ros2_control#165限位咬合); mock/mujoco展开逐字节不变; verify piper --with-gazebo 36全绿

File: unistackbot_description/arms/piper/urdf/piper_ros2_control.xacro (robot description, xacro)
@@ -40,5 +40,15 @@
             <joint name="joint2">
                 <command_interface name="position"/>
-                <state_interface name="position"/>
+                <!-- gz/ODE 已知行为 (上游 gz_ros2_control issue #165): 关节静置恰好压在限位上会被
+                     限位约束咬死, 无法再命令离开 (捕获区微米级, 官方 demo 用 initial_value 规避)。
+                     本关节限位 0..3.14, 启动位 0=下限, 故 ign 链启动即抬 0.01 rad -->
+                <xacro:if value="${use_gazebo == 'ign'}">
+                    <state_interface name="position">
+                        <param name="initial_value">0.01</param>
+                    </state_interface>
+                </xacro:if>
+                <xacro:unless value="${use_gazebo == 'ign'}">
+                    <state_interface name="position"/>
+                </xacro:unless>
                 <state_interface name="velocity"/>
                 <state_interface name="effort"/>
@@ -49,5 +59,13 @@
             <joint name="joint3">
                 <command_interface name="position"/>
-                <state_interface name="position"/>
+                <!-- 同 joint2: 限位 -2.97..0, 启动位 0=上限, ign 链启动即压 -0.01 rad 离开限位线 -->
+                <xacro:if value="${use_gazebo == 'ign'}">
+                    <state_interface name="position">
+                        <param name="initial_value">-0.01</param>
+                    </state_interface>
+                </xacro:if>
+                <xacro:unless value="${use_gazebo == 'ign'}">
+                    <state_interface name="position"/>
+                </xacro:unless>
                 <state_interface name="velocity"/>
                 <state_interface name="effort"/>
@@ -86,5 +104,13 @@
                 <joint name="gripper">
                     <command_interface name="position"/>
-                    <state_interface name="position"/>
+                    <!-- 同 joint2: 限位 0..0.1, 启动位 0=下限, ign 链启动即张 0.001 m (1mm/全程100mm) -->
+                    <xacro:if value="${use_gazebo == 'ign'}">
+                        <state_interface name="position">
+                            <param name="initial_value">0.001</param>
+                        </state_interface>
+                    </xacro:if>
+                    <xacro:unless value="${use_gazebo == 'ign'}">
+                        <state_interface name="position"/>
+                    </xacro:unless>
                     <state_interface name="velocity"/>
                     <param name="min">0</param>
@@ -93,10 +119,10 @@
                 </joint>
                 <!-- 两个 mimic 手指关节, 按链分流:
-                     mujoco/ign: passive —— 无 command_interface, 跟随由仿真侧原生 mimic 语义承担
-                       (mujoco: MJCF equality, 见 mujoco/README.md; gz 0.7.21+: URDF <mimic> 标签,
-                       插件原生处理)。JointStream 解析后只管 7 个主关节。
-                       2026-09-21 实测: gz_ros2_control 升级 0.7.21 后 (mujoco 安装的 apt 连带),
-                       带 mimic 参数声明手指会被导出为 <joint>_mimic 接口名 → JS 声明 9 关节对不上
-                       "Not acceptable command interfaces combination"。
+                     mujoco/ign: passive —— 无 command_interface。mujoco: 跟随由 MJCF equality 承担
+                       (见 mujoco/README.md)。ign: 插件 mimic 只认 ros2_control 块 mimic/multiplier
+                       参数 (0.7.20/0.7.21 相同), URDF <mimic> 标签被 sdformat 转换丢弃 —— 手指实为
+                       自由关节, 已知漂移; 加 mimic 参数可获插件内 P 驱动耦合, 但接口会带 _mimic 后缀
+                       污染 /joint_states 关节名, 耦合方案待裁决 (独立工作项)。
+                       JointStream 解析后只管 7 个主关节。
                      mock/Classic: 按 gazebo_ros2_control 要求补 mimic/multiplier 参数受控跟随 -->
                 <xacro:if value="${use_gazebo in ['mujoco', 'ign']}">

Commit message: 夹爪契约=物理DOF:从指state-only统一命令面

File: unistackbot_description/arms/piper/urdf/piper_ros2_control.xacro (robot description, xacro)
@@ -136,5 +136,6 @@
                     </joint>
                 </xacro:if>
-                <xacro:unless value="${use_gazebo in ['mujoco', 'ign']}">
+                <xacro:if value="${use_gazebo in [True, 'true', 'classic']}">
+                    <!-- classic: gazebo_ros2_control 的 mimic 需命令接口 + 参数 (插件内镜像) -->
                     <joint name="gripper_joint1">
                         <command_interface name="position"/>
@@ -153,5 +154,24 @@
                         <param name="offset">0.0</param>
                     </joint>
-                </xacro:unless>
+                </xacro:if>
+                <xacro:if value="${use_gazebo in [False, 'false']}">
+                    <!-- mock (2026-10-20 契约=物理DOF): 从指 state-only —— 对外命令面 7 关节
+                         (= 真机 SDK 形状, Jazzy+ 原生 mimic 同方向); 耦合由 kinematic backend
+                         按 mimic/multiplier 参数推导 (与 mujoco equality 同构) -->
+                    <joint name="gripper_joint1">
+                        <state_interface name="position"/>
+                        <state_interface name="velocity"/>
+                        <param name="mimic">gripper</param>
+                        <param name="multiplier">0.5</param>
+                        <param name="offset">0.0</param>
+                    </joint>
+                    <joint name="gripper_joint2">
+                        <state_interface name="position"/>
+                        <state_interface name="velocity"/>
+                        <param name="mimic">gripper</param>
+                        <param name="multiplier">-0.5</param>
+                        <param name="offset">0.0</param>
+                    </joint>
+                </xacro:if>
             </xacro:if>
         </ros2_control>

File: unistackbot_description/arms/stationlite/urdf/stationlite_ros2_control.xacro (robot description, xacro)
@@ -47,5 +47,6 @@
             <!-- left_gripper_joint2 (mimic): MuJoCo 模式下 state-only (equality 耦合) -->
             <!-- gripper_joint2 removed for MuJoCo testing -->
-            <xacro:unless value="${use_gazebo == 'mujoco'}">
+            <xacro:if value="${use_gazebo == 'ign'}">
+                <!-- ign: gz 插件 mimic 参数需命令接口 (插件内镜像; _mimic 后缀坑独立挂账) -->
                 <joint name="left_gripper_joint2">
                     <command_interface name="position"/>
@@ -59,5 +60,16 @@
                     <param name="multiplier">-1.0</param>
                 </joint>
-            </xacro:unless>
+            </xacro:if>
+            <xacro:if value="${use_gazebo in [False, 'false']}">
+                <!-- mock (2026-10-20 契约=物理DOF): 从指 state-only —— 命令面 14 关节
+                     (= 真机 SDK setGripperPosition 单值形状); 耦合由 kinematic backend
+                     按 mimic/multiplier 推导 (与 mujoco equality 同构) -->
+                <joint name="left_gripper_joint2">
+                    <state_interface name="position"/>
+                    <state_interface name="velocity"/>
+                    <param name="mimic">left_gripper_joint1</param>
+                    <param name="multiplier">-1.0</param>
+                </joint>
+            </xacro:if>
             <!-- 右臂 6 关节 (与左臂对称) -->
             <xacro:stationlite_revolute_joint joint_name="right_joint1" lo="-2.824" hi="2.824" effort="10" vel="3.0"/>
@@ -79,5 +91,6 @@
             <!-- right_gripper_joint2 (mimic): MuJoCo 模式下 state-only -->
             <!-- gripper_joint2 removed for MuJoCo testing -->
-            <xacro:unless value="${use_gazebo == 'mujoco'}">
+            <xacro:if value="${use_gazebo == 'ign'}">
+                <!-- ign: gz 插件 mimic 参数需命令接口 (插件内镜像; _mimic 后缀坑独立挂账) -->
                 <joint name="right_gripper_joint2">
                     <command_interface name="position"/>
@@ -91,5 +104,16 @@
                     <param name="multiplier">-1.0</param>
                 </joint>
-            </xacro:unless>
+            </xacro:if>
+            <xacro:if value="${use_gazebo in [False, 'false']}">
+                <!-- mock (2026-10-20 契约=物理DOF): 从指 state-only —— 命令面 14 关节
+                     (= 真机 SDK setGripperPosition 单值形状); 耦合由 kinematic backend
+                     按 mimic/multiplier 推导 (与 mujoco equality 同构) -->
+                <joint name="right_gripper_joint2">
+                    <state_interface name="position"/>
+                    <state_interface name="velocity"/>
+                    <param name="mimic">right_gripper_joint1</param>
+                    <param name="multiplier">-1.0</param>
+                </joint>
+            </xacro:if>
         </ros2_control>
     </xacro:macro>
