Commit message: 新增 Gazebo 仿真集成,控制器切换为 JTC
- 新增 unistackbot_gazebo 包(empty world + gazebo.launch.py)
- piper_controllers.yaml 由 ForwardCommandController 改为 JointTrajectoryController
- piper_control.launch.py 添加控制器 spawner
- xacro 新增 use_gazebo 参数,切换 GazeboSystem / MockPiperHardware 插件
- piper_macro.xacro 修复 parent 为 base_link 时重复关节的问题

Co-Authored-By: Claude Opus 4.7 <noreply@anthropic.com>

File: unistackbot_description/arms/piper/urdf/piper.urdf.xacro (robot description, xacro)
@@ -4,4 +4,5 @@
     <xacro:arg name="use_ros2_control" default="false" />
     <xacro:arg name="use_world" default="true" />
+    <xacro:arg name="use_gazebo" default="false" />
     <xacro:include filename="$(find unistackbot_description)/arms/piper/urdf/piper_macro.xacro"/>
     <xacro:include filename="$(find unistackbot_description)/arms/piper/urdf/piper_gripper_macro.xacro"/>
@@ -18,5 +19,12 @@
     </xacro:if>
     <xacro:if value="$(arg use_ros2_control)">
-        <xacro:piper_ros2_control use_gripper="$(arg use_gripper)"/>
+        <xacro:piper_ros2_control use_gripper="$(arg use_gripper)" use_gazebo="$(arg use_gazebo)"/>
+    </xacro:if>
+    <xacro:if value="$(arg use_gazebo)">
+        <gazebo>
+            <plugin name="gazebo_ros2_control" filename="libgazebo_ros2_control.so">
+                <parameters>$(find unistackbot_bringup)/config/piper_controllers.yaml</parameters>
+            </plugin>
+        </gazebo>
     </xacro:if>
 </robot>

File: unistackbot_description/arms/piper/urdf/piper_macro.xacro (robot description, xacro)
@@ -2,9 +2,11 @@
 <robot xmlns:xacro="http://www.ros.org/wiki/xacro">
     <xacro:macro name="piper_arm" params="parent:=base_link origin_xyz:='0 0 0' origin_rpy:='0 0 0'">
-        <joint name="world_to_base_link" type="fixed">
-            <parent link="${parent}"/>
-            <child link="base_link"/>
-            <origin xyz="${origin_xyz}" rpy="${origin_rpy}"/>
-        </joint>
+        <xacro:unless value="${parent == 'base_link'}">
+            <joint name="world_to_base_link" type="fixed">
+                <parent link="${parent}"/>
+                <child link="base_link"/>
+                <origin xyz="${origin_xyz}" rpy="${origin_rpy}"/>
+            </joint>
+        </xacro:unless>
         <link name="base_link">
             <inertial>

File: unistackbot_description/arms/piper/urdf/piper_ros2_control.xacro (robot description, xacro)
@@ -1,8 +1,13 @@
 <?xml version="1.0" encoding="utf-8"?>
 <robot xmlns:xacro="http://www.ros.org/wiki/xacro">
-    <xacro:macro name="piper_ros2_control" params="use_gripper:=true">
+    <xacro:macro name="piper_ros2_control" params="use_gripper:=true use_gazebo:=false">
         <ros2_control name="piper_system" type="system">
             <hardware>
-                <plugin>unistackbot_hardware_mock/MockPiperHardware</plugin>
+                <xacro:if value="${use_gazebo}">
+                    <plugin>gazebo_ros2_control/GazeboSystem</plugin>
+                </xacro:if>
+                <xacro:unless value="${use_gazebo}">
+                    <plugin>unistackbot_hardware_mock/MockPiperHardware</plugin>
+                </xacro:unless>
                 <param name="device">/dev/piper_arm</param>
                 <param name="baudrate">2000000</param>

Commit message: 迁移 Gazebo Fortress 并打通仿真控制链路
Co-Authored-By: Claude <noreply@anthropic.com>

File: unistackbot_description/arms/piper/urdf/piper.urdf.xacro (robot description, xacro)
@@ -21,10 +21,3 @@
         <xacro:piper_ros2_control use_gripper="$(arg use_gripper)" use_gazebo="$(arg use_gazebo)"/>
     </xacro:if>
-    <xacro:if value="$(arg use_gazebo)">
-        <gazebo>
-            <plugin name="gazebo_ros2_control" filename="libgazebo_ros2_control.so">
-                <parameters>$(find unistackbot_bringup)/config/piper_controllers.yaml</parameters>
-            </plugin>
-        </gazebo>
-    </xacro:if>
 </robot>

File: unistackbot_description/arms/piper/urdf/piper_gripper_macro.xacro (robot description, xacro)
@@ -50,5 +50,13 @@
             <child link="gripper_base"/>
         </joint>
-        <link name="gripper_link"/>
+        <!-- gripper_link 必须带惯性: 空 link 会被 Gazebo 丢弃, 导致 gripper 关节
+             在仿真中不存在, JTC 因缺关节无法激活 -->
+        <link name="gripper_link">
+            <inertial>
+                <origin xyz="0 0 0.01" rpy="0 0 0"/>
+                <mass value="0.01"/>
+                <inertia ixx="1e-06" ixy="0.0" ixz="0.0" iyy="1e-06" iyz="0.0" izz="1e-06"/>
+            </inertial>
+        </link>
         <joint name="gripper" type="prismatic">
             <origin xyz="0 0 0" rpy="0 0 0"/>

File: unistackbot_description/arms/piper/urdf/piper_ros2_control.xacro (robot description, xacro)
@@ -4,8 +4,13 @@
         <ros2_control name="piper_system" type="system">
             <hardware>
-                <xacro:if value="${use_gazebo}">
+                <!-- use_gazebo: 'ign'=Gazebo Sim(Fortress), 'true'/'classic'=Gazebo Classic, 其余=mock 插件.
+                     注意: $(arg) 传参时 xacro 会把 true/false 解析成 Python 布尔, 条件需同时匹配 True -->
+                <xacro:if value="${use_gazebo == 'ign'}">
+                    <plugin>gz_ros2_control/GazeboSimSystem</plugin>
+                </xacro:if>
+                <xacro:if value="${use_gazebo in [True, 'true', 'classic']}">
                     <plugin>gazebo_ros2_control/GazeboSystem</plugin>
                 </xacro:if>
-                <xacro:unless value="${use_gazebo}">
+                <xacro:unless value="${use_gazebo in ['ign', True, 'true', 'classic']}">
                     <plugin>unistackbot_hardware_mock/MockPiperHardware</plugin>
                 </xacro:unless>
@@ -62,5 +67,5 @@
                 <param name="max">2.0943951</param>
             </joint>
-            <xacro:if value="$(arg use_gripper)">
+            <xacro:if value="${use_gripper}">
                 <joint name="gripper">
                     <command_interface name="position"/>
@@ -70,6 +75,41 @@
                     <param name="max">0.1</param>
                 </joint>
+                <!-- 两个 mimic 手指关节: URDF 侧已有 <mimic> 标签, 此处按 gazebo_ros2_control
+                     要求补 mimic/multiplier 参数才能在仿真中受控跟随 gripper -->
+                <joint name="gripper_joint1">
+                    <command_interface name="position"/>
+                    <state_interface name="position"/>
+                    <state_interface name="velocity"/>
+                    <param name="mimic">gripper</param>
+                    <param name="multiplier">0.5</param>
+                    <param name="offset">0.0</param>
+                </joint>
+                <joint name="gripper_joint2">
+                    <command_interface name="position"/>
+                    <state_interface name="position"/>
+                    <state_interface name="velocity"/>
+                    <param name="mimic">gripper</param>
+                    <param name="multiplier">-0.5</param>
+                    <param name="offset">0.0</param>
+                </joint>
             </xacro:if>
         </ros2_control>
+        <!-- Gazebo 侧系统插件: 与上方 use_gazebo 模式对应, 控制器配置共用 bringup 的 yaml -->
+        <xacro:if value="${use_gazebo in [True, 'true', 'classic']}">
+            <gazebo>
+                <plugin name="gazebo_ros2_control" filename="libgazebo_ros2_control.so">
+                    <parameters>$(find unistackbot_bringup)/config/piper_controllers.yaml</parameters>
+                </plugin>
+            </gazebo>
+        </xacro:if>
+        <xacro:if value="${use_gazebo == 'ign'}">
+            <gazebo>
+                <plugin filename="gz_ros2_control-system" name="gz_ros2_control::GazeboSimROS2ControlPlugin">
+                    <robot_param>robot_description</robot_param>
+                    <robot_param_node>robot_state_publisher</robot_param_node>
+                    <parameters>$(find unistackbot_bringup)/config/piper_controllers.yaml</parameters>
+                </plugin>
+            </gazebo>
+        </xacro:if>
     </xacro:macro>
 </robot>
