Commit message: xarm7 MJCF资产+mujoco四路分支: MuJoCo链双机型全绿(跟踪1.0mrad/CM收敛0.68mm, damping取URDF厂商值零接触无需exclude)

File: unistackbot_description/arms/xarm7/urdf/xarm7.urdf.xacro (robot description, xacro)
@@ -4,4 +4,6 @@
     <xacro:arg name="use_world" default="true" />
     <xacro:arg name="use_gazebo" default="false" />
+    <!-- mujoco 链: 是否无头 (不拉 Simulate 渲染窗); 传给 ros2_control 块的 headless 硬件参数 -->
+    <xacro:arg name="headless" default="true" />
     <!-- 全局属性: 上游 common 宏依赖(mesh 路径前缀/后缀, YAML 加载方式) -->
     <xacro:property name="mesh_path" value="package://unistackbot_description/arms/xarm7/meshes" />
@@ -24,5 +26,5 @@
         kinematics_params_filename="$(find unistackbot_description)/arms/xarm7/config/kinematics/default/xarm7_default_kinematics.yaml"/>
     <xacro:if value="$(arg use_ros2_control)">
-        <xacro:xarm7_ros2_control use_gazebo="$(arg use_gazebo)"/>
+        <xacro:xarm7_ros2_control use_gazebo="$(arg use_gazebo)" headless="$(arg headless)"/>
     </xacro:if>
 </robot>

File: unistackbot_description/arms/xarm7/urdf/xarm7_ros2_control.xacro (robot description, xacro)
@@ -1,16 +1,25 @@
 <?xml version="1.0" encoding="utf-8"?>
 <robot xmlns:xacro="http://www.ros.org/wiki/xacro">
-    <xacro:macro name="xarm7_ros2_control" params="use_gazebo:=false">
+    <xacro:macro name="xarm7_ros2_control" params="use_gazebo:=false headless:=true">
         <ros2_control name="xarm7_system" type="system">
             <hardware>
-                <!-- use_gazebo: 'ign'=Gazebo Sim(Fortress), 'true'/'classic'=Gazebo Classic, 其余=mock 插件.
+                <!-- use_gazebo: 'ign'=Gazebo Sim(Fortress), 'mujoco'=MuJoCo(mujoco_ros2_control),
+                     'true'/'classic'=Gazebo Classic, 其余=mock 插件.
                      注意: $(arg) 传参时 xacro 会把 true/false 解析成 Python 布尔, 条件需同时匹配 True -->
                 <xacro:if value="${use_gazebo == 'ign'}">
                     <plugin>gz_ros2_control/GazeboSimSystem</plugin>
                 </xacro:if>
+                <xacro:if value="${use_gazebo == 'mujoco'}">
+                    <plugin>mujoco_ros2_control/MujocoSystemInterface</plugin>
+                    <!-- MJCF 资产: 身体树由本 URDF 转换 + 手工策展, 见 arms/xarm7/mujoco/README.md -->
+                    <param name="mujoco_model">$(find unistackbot_description)/arms/xarm7/mujoco/xarm7.xml</param>
+                    <param name="sim_speed_factor">1.0</param>
+                    <!-- $(arg) 布尔坑: true 会变成 Python True, 归一回小写字符串 -->
+                    <param name="headless">${'true' if headless in [True, 'true'] else 'false'}</param>
+                </xacro:if>
                 <xacro:if value="${use_gazebo in [True, 'true', 'classic']}">
                     <plugin>gazebo_ros2_control/GazeboSystem</plugin>
                 </xacro:if>
-                <xacro:unless value="${use_gazebo in ['ign', True, 'true', 'classic']}">
+                <xacro:unless value="${use_gazebo in ['ign', 'mujoco', True, 'true', 'classic']}">
                     <plugin>unistackbot_sim_control/SimControlHardware</plugin>
                     <param name="backend">kinematic</param>
