Commit message: 修stationlite mesh路径加visual子目录

File: unistackbot_description/arms/stationlite/urdf/stationlite_macro.xacro (robot description, xacro)
@@ -12,5 +12,5 @@
       <visual>
         <origin xyz="0 0 0" rpy="0 0 0"/>
-        <geometry><mesh filename="package://unistackbot_description/arms/stationlite/meshes/base.STL"/></geometry>
+        <geometry><mesh filename="package://unistackbot_description/arms/stationlite/meshes/visual/base.STL"/></geometry>
         <material name="station_gray"/>
       </visual>
@@ -24,5 +24,5 @@
       <visual>
         <origin xyz="0 0 0" rpy="0 0 0"/>
-        <geometry><mesh filename="package://unistackbot_description/arms/stationlite/meshes/armbase.STL"/></geometry>
+        <geometry><mesh filename="package://unistackbot_description/arms/stationlite/meshes/visual/armbase.STL"/></geometry>
         <material name="station_gray"/>
       </visual>
@@ -36,5 +36,5 @@
       <visual>
         <origin xyz="0 0 0" rpy="0 0 0"/>
-        <geometry><mesh filename="package://unistackbot_description/arms/stationlite/meshes/link1.STL"/></geometry>
+        <geometry><mesh filename="package://unistackbot_description/arms/stationlite/meshes/visual/link1.STL"/></geometry>
         <material name="station_gray"/>
       </visual>
@@ -48,5 +48,5 @@
       <visual>
         <origin xyz="0 0 0" rpy="0 0 0"/>
-        <geometry><mesh filename="package://unistackbot_description/arms/stationlite/meshes/link2.STL"/></geometry>
+        <geometry><mesh filename="package://unistackbot_description/arms/stationlite/meshes/visual/link2.STL"/></geometry>
         <material name="station_gray"/>
       </visual>
@@ -60,5 +60,5 @@
       <visual>
         <origin xyz="0 0 0" rpy="0 0 0"/>
-        <geometry><mesh filename="package://unistackbot_description/arms/stationlite/meshes/link3.STL"/></geometry>
+        <geometry><mesh filename="package://unistackbot_description/arms/stationlite/meshes/visual/link3.STL"/></geometry>
         <material name="station_gray"/>
       </visual>
@@ -72,5 +72,5 @@
       <visual>
         <origin xyz="0 0 0" rpy="0 0 0"/>
-        <geometry><mesh filename="package://unistackbot_description/arms/stationlite/meshes/link4.STL"/></geometry>
+        <geometry><mesh filename="package://unistackbot_description/arms/stationlite/meshes/visual/link4.STL"/></geometry>
         <material name="station_gray"/>
       </visual>
@@ -84,5 +84,5 @@
       <visual>
         <origin xyz="0 0 0" rpy="0 0 0"/>
-        <geometry><mesh filename="package://unistackbot_description/arms/stationlite/meshes/link5.STL"/></geometry>
+        <geometry><mesh filename="package://unistackbot_description/arms/stationlite/meshes/visual/link5.STL"/></geometry>
         <material name="station_gray"/>
       </visual>
@@ -96,5 +96,5 @@
       <visual>
         <origin xyz="0 0 0" rpy="0 0 0"/>
-        <geometry><mesh filename="package://unistackbot_description/arms/stationlite/meshes/gripper_base.STL"/></geometry>
+        <geometry><mesh filename="package://unistackbot_description/arms/stationlite/meshes/visual/gripper_base.STL"/></geometry>
         <material name="station_gray"/>
       </visual>
@@ -108,5 +108,5 @@
       <visual>
         <origin xyz="0 0 0" rpy="0 0 0"/>
-        <geometry><mesh filename="package://unistackbot_description/arms/stationlite/meshes/griperlj_link1.STL"/></geometry>
+        <geometry><mesh filename="package://unistackbot_description/arms/stationlite/meshes/visual/griperlj_link1.STL"/></geometry>
         <material name="station_gray"/>
       </visual>
@@ -120,5 +120,5 @@
       <visual>
         <origin xyz="0 0 0" rpy="0 0 0"/>
-        <geometry><mesh filename="package://unistackbot_description/arms/stationlite/meshes/griperlj_link2.STL"/></geometry>
+        <geometry><mesh filename="package://unistackbot_description/arms/stationlite/meshes/visual/griperlj_link2.STL"/></geometry>
         <material name="station_gray"/>
       </visual>
@@ -132,5 +132,5 @@
       <visual>
         <origin xyz="0 0 0" rpy="0 0 0"/>
-        <geometry><mesh filename="package://unistackbot_description/arms/stationlite/meshes/handcam.STL"/></geometry>
+        <geometry><mesh filename="package://unistackbot_description/arms/stationlite/meshes/visual/handcam.STL"/></geometry>
         <material name="station_gray"/>
       </visual>
@@ -211,5 +211,5 @@
       <visual>
         <origin xyz="0 0 0" rpy="0 0 0"/>
-        <geometry><mesh filename="package://unistackbot_description/arms/stationlite/meshes/armbase.STL"/></geometry>
+        <geometry><mesh filename="package://unistackbot_description/arms/stationlite/meshes/visual/armbase.STL"/></geometry>
         <material name="station_gray"/>
       </visual>
@@ -223,5 +223,5 @@
       <visual>
         <origin xyz="0 0 0" rpy="0 0 0"/>
-        <geometry><mesh filename="package://unistackbot_description/arms/stationlite/meshes/link1.STL"/></geometry>
+        <geometry><mesh filename="package://unistackbot_description/arms/stationlite/meshes/visual/link1.STL"/></geometry>
         <material name="station_gray"/>
       </visual>
@@ -235,5 +235,5 @@
       <visual>
         <origin xyz="0 0 0" rpy="0 0 0"/>
-        <geometry><mesh filename="package://unistackbot_description/arms/stationlite/meshes/link2.STL"/></geometry>
+        <geometry><mesh filename="package://unistackbot_description/arms/stationlite/meshes/visual/link2.STL"/></geometry>
         <material name="station_gray"/>
       </visual>
@@ -247,5 +247,5 @@
       <visual>
         <origin xyz="0 0 0" rpy="0 0 0"/>
-        <geometry><mesh filename="package://unistackbot_description/arms/stationlite/meshes/link3.STL"/></geometry>
+        <geometry><mesh filename="package://unistackbot_description/arms/stationlite/meshes/visual/link3.STL"/></geometry>
         <material name="station_gray"/>
       </visual>
@@ -259,5 +259,5 @@
       <visual>
         <origin xyz="0 0 0" rpy="0 0 0"/>
-        <geometry><mesh filename="package://unistackbot_description/arms/stationlite/meshes/link4.STL"/></geometry>
+        <geometry><mesh filename="package://unistackbot_description/arms/stationlite/meshes/visual/link4.STL"/></geometry>
         <material name="station_gray"/>
       </visual>
@@ -271,5 +271,5 @@
       <visual>
         <origin xyz="0 0 0" rpy="0 0 0"/>
-        <geometry><mesh filename="package://unistackbot_description/arms/stationlite/meshes/link5.STL"/></geometry>
+        <geometry><mesh filename="package://unistackbot_description/arms/stationlite/meshes/visual/link5.STL"/></geometry>
         <material name="station_gray"/>
       </visual>
@@ -283,5 +283,5 @@
       <visual>
         <origin xyz="0 0 0" rpy="0 0 0"/>
-        <geometry><mesh filename="package://unistackbot_description/arms/stationlite/meshes/gripper_base.STL"/></geometry>
+        <geometry><mesh filename="package://unistackbot_description/arms/stationlite/meshes/visual/gripper_base.STL"/></geometry>
         <material name="station_gray"/>
       </visual>
@@ -295,5 +295,5 @@
       <visual>
         <origin xyz="0 0 0" rpy="0 0 0"/>
-        <geometry><mesh filename="package://unistackbot_description/arms/stationlite/meshes/griperlj_link1.STL"/></geometry>
+        <geometry><mesh filename="package://unistackbot_description/arms/stationlite/meshes/visual/griperlj_link1.STL"/></geometry>
         <material name="station_gray"/>
       </visual>
@@ -307,5 +307,5 @@
       <visual>
         <origin xyz="0 0 0" rpy="0 0 0"/>
-        <geometry><mesh filename="package://unistackbot_description/arms/stationlite/meshes/griperlj_link2.STL"/></geometry>
+        <geometry><mesh filename="package://unistackbot_description/arms/stationlite/meshes/visual/griperlj_link2.STL"/></geometry>
         <material name="station_gray"/>
       </visual>
@@ -319,5 +319,5 @@
       <visual>
         <origin xyz="0 0 0" rpy="0 0 0"/>
-        <geometry><mesh filename="package://unistackbot_description/arms/stationlite/meshes/handcam.STL"/></geometry>
+        <geometry><mesh filename="package://unistackbot_description/arms/stationlite/meshes/visual/handcam.STL"/></geometry>
         <material name="station_gray"/>
       </visual>

Commit message: 补stationlite material定义

File: unistackbot_description/arms/stationlite/urdf/stationlite_macro.xacro (robot description, xacro)
@@ -1,4 +1,7 @@
 <?xml version="1.0" encoding="utf-8"?>
 <robot xmlns:xacro="http://www.ros.org/wiki/xacro">
+  <material name="station_gray">
+    <color rgba="0.75294 0.75294 0.75294 1"/>
+  </material>
   <!-- stationlite 双臂 macro: base + 左右对称 6-DOF + 平移夹爪 -->
   <!-- 资产来源: Lumos Station Lite 原始 URDF (arms/stationlite/original/) -->
