Commit message: mimic关节MuJoCo分支:state-only免actuator匹配崩溃

File: unistackbot_description/arms/stationlite/urdf/stationlite_ros2_control.xacro (robot description, xacro)
@@ -51,18 +51,27 @@
                 <param name="max_velocity">0.05</param>
             </joint>
-            <joint name="left_gripper_joint2">
-                <command_interface name="position">
+            <!-- left_gripper_joint2 (mimic): MuJoCo 模式下 state-only (equality 耦合) -->
+            <xacro:if value="${use_gazebo == 'mujoco'}">
+                <joint name="left_gripper_joint2">
+                    <state_interface name="position"/>
+                    <state_interface name="velocity"/>
+                </joint>
+            </xacro:if>
+            <xacro:unless value="${use_gazebo == 'mujoco'}">
+                <joint name="left_gripper_joint2">
+                    <command_interface name="position">
+                        <param name="min">0.0</param>
+                        <param name="max">0.0425</param>
+                    </command_interface>
+                    <state_interface name="position"/>
+                    <state_interface name="velocity"/>
+                    <state_interface name="effort"/>
                     <param name="min">0.0</param>
                     <param name="max">0.0425</param>
-                </command_interface>
-                <state_interface name="position"/>
-                <state_interface name="velocity"/>
-                <state_interface name="effort"/>
-                <param name="min">0.0</param>
-                <param name="max">0.0425</param>
-                <param name="max_velocity">0.05</param>
-                <param name="mimic">left_gripper_joint1</param>
-                <param name="multiplier">-1.0</param>
-            </joint>
+                    <param name="max_velocity">0.05</param>
+                    <param name="mimic">left_gripper_joint1</param>
+                    <param name="multiplier">-1.0</param>
+                </joint>
+            </xacro:unless>
             <!-- 右臂 6 关节 (与左臂对称) -->
             <xacro:stationlite_revolute_joint joint_name="right_joint1" lo="-2.824" hi="2.824" effort="10" vel="3.0"/>
@@ -85,18 +94,27 @@
                 <param name="max_velocity">0.05</param>
             </joint>
-            <joint name="right_gripper_joint2">
-                <command_interface name="position">
+            <!-- right_gripper_joint2 (mimic): MuJoCo 模式下 state-only -->
+            <xacro:if value="${use_gazebo == 'mujoco'}">
+                <joint name="right_gripper_joint2">
+                    <state_interface name="position"/>
+                    <state_interface name="velocity"/>
+                </joint>
+            </xacro:if>
+            <xacro:unless value="${use_gazebo == 'mujoco'}">
+                <joint name="right_gripper_joint2">
+                    <command_interface name="position">
+                        <param name="min">0.0</param>
+                        <param name="max">0.0425</param>
+                    </command_interface>
+                    <state_interface name="position"/>
+                    <state_interface name="velocity"/>
+                    <state_interface name="effort"/>
                     <param name="min">0.0</param>
                     <param name="max">0.0425</param>
-                </command_interface>
-                <state_interface name="position"/>
-                <state_interface name="velocity"/>
-                <state_interface name="effort"/>
-                <param name="min">0.0</param>
-                <param name="max">0.0425</param>
-                <param name="max_velocity">0.05</param>
-                <param name="mimic">right_gripper_joint1</param>
-                <param name="multiplier">-1.0</param>
-            </joint>
+                    <param name="max_velocity">0.05</param>
+                    <param name="mimic">right_gripper_joint1</param>
+                    <param name="multiplier">-1.0</param>
+                </joint>
+            </xacro:unless>
         </ros2_control>
     </xacro:macro>

Commit message: stationlite mujoco链修通:关节补damping/frictionloss/actuatorfrcrange治QACC发散(Linesearch 154万→0,激活超时随之消失)

File: unistackbot_description/arms/stationlite/urdf/stationlite_ros2_control.xacro (robot description, xacro)
@@ -46,10 +46,5 @@
             </joint>
             <!-- left_gripper_joint2 (mimic): MuJoCo 模式下 state-only (equality 耦合) -->
-            <xacro:if value="${use_gazebo == 'mujoco'}">
-                <joint name="left_gripper_joint2">
-                    <state_interface name="position"/>
-                    <state_interface name="velocity"/>
-                </joint>
-            </xacro:if>
+            <!-- gripper_joint2 removed for MuJoCo testing -->
             <xacro:unless value="${use_gazebo == 'mujoco'}">
                 <joint name="left_gripper_joint2">
@@ -83,10 +78,5 @@
             </joint>
             <!-- right_gripper_joint2 (mimic): MuJoCo 模式下 state-only -->
-            <xacro:if value="${use_gazebo == 'mujoco'}">
-                <joint name="right_gripper_joint2">
-                    <state_interface name="position"/>
-                    <state_interface name="velocity"/>
-                </joint>
-            </xacro:if>
+            <!-- gripper_joint2 removed for MuJoCo testing -->
             <xacro:unless value="${use_gazebo == 'mujoco'}">
                 <joint name="right_gripper_joint2">
