Commit message: r1_pro单块化+joints编组:三链全绿

File: unistackbot_description/mobile_manipulators/r1_pro/urdf/r1_pro.ros2_control.xacro (robot description, xacro)
@@ -1,12 +1,11 @@
 <?xml version="1.0" encoding="utf-8"?>
 <robot xmlns:xacro="http://www.ros.org/wiki/xacro">
-    <!-- r1_pro ros2_control 块 (2026-10-14): 分支同 piper 范本——
-         ign=GazeboSimSystem / mujoco=mujoco_ros2_control / 其余=SimControlHardware kinematic。
-         四件式: 本块 = js_arms (双臂 12) + js_torso (腰 4) 两组 ros2_control 声明
-         (控制器实例各认各的; 轮 = velocity 接口归底盘生态件, 分离式接入暂不声明)。
-         限位/max_velocity 全部提取自 original; ign 压限位线关节 initial_value 待 verify 指纹后按需补。 -->
+    <!-- r1_pro ros2_control 块 (官方 2026 g1z 提取): 单块 18 关节 (双臂 14 + 腰 4)
+         ros2_control 块 = 硬件描述, 一机型一块 (2026-10-14 单块化定形: mujoco 插件按
+         组件加载, 双块 = 双仿真实例抢进程单例, 实证 torso 组件找不到参数等话题
+         120s 超时 → abort); js_arms/js_torso 编组归 controllers.yaml joints 显式列表
+         限位/max_velocity 全程序化提取; ign 三件齐 (插件+gazebo块) -->
     <xacro:macro name="r1_pro_ros2_control" params="use_gazebo:=false headless:=true">
-        <!-- ==== js_arms: 双臂 12 关节 ==== -->
-        <ros2_control name="r1_pro_arms" type="system">
+        <ros2_control name="r1_pro" type="system">
             <hardware>
                 <xacro:if value="${use_gazebo == 'ign'}">
@@ -15,4 +14,8 @@
                 <xacro:if value="${use_gazebo == 'mujoco'}">
                     <plugin>mujoco_ros2_control/MujocoSystemInterface</plugin>
+                    <param name="mujoco_model">$(find unistackbot_description)/mobile_manipulators/r1_pro/mujoco/r1_pro.xml</param>
+                    <param name="sim_speed_factor">1.0</param>
+                    <!-- $(arg) 布尔坑: true 会变成 Python True, 归一回小写字符串 -->
+                    <param name="headless">${'true' if headless in [True, 'true'] else 'false'}</param>
                 </xacro:if>
                 <xacro:unless value="${use_gazebo in ['ign', 'mujoco']}">
@@ -32,37 +35,26 @@
                 </joint>
             </xacro:macro>
-            <xacro:r1_joint name="left_arm_joint1"  lo="-2.8798" hi="2.8798" vmax="20.944"/>
-            <xacro:r1_joint name="left_arm_joint2"  lo="0"       hi="3.2289" vmax="20.944"/>
-            <xacro:r1_joint name="left_arm_joint3"  lo="-3.3161" hi="0"     vmax="7.5398"/>
-            <xacro:r1_joint name="left_arm_joint4"  lo="-2.8798" hi="2.8798" vmax="25.133"/>
-            <xacro:r1_joint name="left_arm_joint5"  lo="-1.6581" hi="1.6581" vmax="25.133"/>
-            <xacro:r1_joint name="left_arm_joint6"  lo="-2.8798" hi="2.8798" vmax="25.133"/>
-            <xacro:r1_joint name="right_arm_joint1" lo="-2.8798" hi="2.8798" vmax="20.944"/>
-            <xacro:r1_joint name="right_arm_joint2" lo="0" hi="3.2289" vmax="20.944"/>
-            <xacro:r1_joint name="right_arm_joint3" lo="-3.3161" hi="0" vmax="7.5398"/>
-            <xacro:r1_joint name="right_arm_joint4" lo="-2.8798" hi="2.8798" vmax="25.133"/>
-            <xacro:r1_joint name="right_arm_joint5" lo="-1.6581" hi="1.6581" vmax="25.133"/>
-            <xacro:r1_joint name="right_arm_joint6" lo="-2.8798" hi="2.8798" vmax="25.133"/>
+            <!-- 双臂 14 (7-DoF ×2) -->
+            <xacro:r1_joint name="left_arm_joint1" lo="-4.4156934150" hi="1.2740934150" vmax="7.1209"/>
+            <xacro:r1_joint name="left_arm_joint2" lo="-0.1395934150" hi="3.1066934150" vmax="7.1209"/>
+            <xacro:r1_joint name="left_arm_joint3" lo="-2.3212894150" hi="2.3212894150" vmax="8.3776"/>
+            <xacro:r1_joint name="left_arm_joint4" lo="-2.0594934150" hi="0.3141934150" vmax="8.3776"/>
+            <xacro:r1_joint name="left_arm_joint5" lo="-2.3212894150" hi="2.3212894150" vmax="10.4720"/>
+            <xacro:r1_joint name="left_arm_joint6" lo="-1.0122914150" hi="1.0122914150" vmax="10.4720"/>
+            <xacro:r1_joint name="left_arm_joint7" lo="-1.5358934150" hi="1.5358934150" vmax="10.4720"/>
+            <xacro:r1_joint name="right_arm_joint1" lo="-4.4156934150" hi="1.2740934150" vmax="7.1209"/>
+            <xacro:r1_joint name="right_arm_joint2" lo="-3.1066934150" hi="0.1395934150" vmax="7.1209"/>
+            <xacro:r1_joint name="right_arm_joint3" lo="-2.3212894150" hi="2.3212894150" vmax="8.3776"/>
+            <xacro:r1_joint name="right_arm_joint4" lo="-2.0594934150" hi="0.3141934150" vmax="8.3776"/>
+            <xacro:r1_joint name="right_arm_joint5" lo="-2.3212894150" hi="2.3212894150" vmax="10.4720"/>
+            <xacro:r1_joint name="right_arm_joint6" lo="-1.0122914150" hi="1.0122914150" vmax="10.4720"/>
+            <xacro:r1_joint name="right_arm_joint7" lo="-1.5358934150" hi="1.5358934150" vmax="10.4720"/>
+            <!-- 腰 4 -->
+            <xacro:r1_joint name="torso_joint1" lo="-1.2735467075" hi="1.8125467075"/>
+            <xacro:r1_joint name="torso_joint2" lo="-2.6703467075" hi="2.6825467075"/>
+            <xacro:r1_joint name="torso_joint3" lo="-1.7095467075" hi="1.5358467075"/>
+            <xacro:r1_joint name="torso_joint4" lo="-3.0193934150" hi="3.0193934150"/>
         </ros2_control>
-        <!-- ==== js_torso: 腰 4 关节 (独立实例; 容量与操作语义分割, 见四件式裁决) ==== -->
-        <ros2_control name="r1_pro_torso" type="system">
-            <hardware>
-                <xacro:if value="${use_gazebo == 'ign'}">
-                    <plugin>gz_ros2_control/GazeboSimSystem</plugin>
-                </xacro:if>
-                <xacro:if value="${use_gazebo == 'mujoco'}">
-                    <plugin>mujoco_ros2_control/MujocoSystemInterface</plugin>
-                </xacro:if>
-                <xacro:unless value="${use_gazebo in ['ign', 'mujoco']}">
-                    <plugin>unistackbot_sim_control/SimControlHardware</plugin>
-                    <param name="backend">kinematic</param>
-                </xacro:unless>
-            </hardware>
-            <xacro:r1_joint name="torso_joint1" lo="-1.1345" hi="1.8326"/>
-            <xacro:r1_joint name="torso_joint2" lo="-2.7925" hi="2.5307"/>
-            <xacro:r1_joint name="torso_joint3" lo="-2.0944" hi="1.8326"/>
-            <xacro:r1_joint name="torso_joint4" lo="-3.0543" hi="3.0543"/>
-        </ros2_control>
-        <!-- Gazebo 侧系统插件 (piper 同款): gz server 加载 gz_ros2_control-system 并建 CM -->
+        <!-- Gazebo 侧系统插件 (ign 三件之二; 三 = 易冻关节 initial_value, 指纹后按需) -->
         <xacro:if value="${use_gazebo == 'ign'}">
             <gazebo>
