Commit message: r1_pro单块化+joints编组:三链全绿

File: unistackbot_description/mobile_manipulators/r1_pro/urdf/r1_pro_macro.xacro (robot description, xacro)
@@ -1,15 +1,17 @@
 <?xml version="1.0" encoding="utf-8"?>
 <robot xmlns:xacro="http://www.ros.org/wiki/xacro">
-    <!-- r1_pro 运动学宏 —— 程序化提取自 original/r1_pro.urdf (2026-10-14, 数字零手抄)
-         覆盖控制域: 腰 torso×4 + 双臂 arm×6×2 = 16 关节 (四件式: js_torso + js_arms)
-         轮 (servo+wheel×3) 与传感器挂点不在此宏 (分离式接入: 底盘生态件, 未驱动时省略) -->
+    <!-- r1_pro 运动学宏 —— 程序化提取自 official urdf_r1pro_g1z_2026 (2026-10-14, 数字零手抄)
+         官方 R1 Pro = 双 7-DoF 臂 + 4-DoF 旋转腰 + 三轮独立转向 (steer+wheel_motor) + g1z 双指爪
+         覆盖控制域 18 关节 = js_torso(4) + js_arms(14, 各自 ≤16 容量内)
+         轮 (steer×3 + wheel_motor×3) / 夹爪 / 传感器挂点不在此宏 (分离式接入) -->
     <xacro:macro name="r1_pro_body">
         <link name="base_link">
             <inertial>
-                <origin xyz="-0.0030503 -0.00009624 0.14087" rpy="0 0 0"/>
-                <mass value="68.732"/>
+                <origin xyz="-0.049262 -0.00008805 0.18255" rpy="0 0 0"/>
+                <mass value="47.63"/>
                 <inertia ixx="1.5812" ixy="-0.00001063" ixz="0.053601" iyy="1.4648" iyz="0.00000571" izz="2.835"/>
             </inertial>
             <visual>
+                <origin xyz="0 0 0" rpy="0 0 0"/>
                 <geometry><mesh filename="package://unistackbot_description/mobile_manipulators/r1_pro/meshes/base_link.STL"/></geometry>
             </visual>
@@ -17,12 +19,12 @@
         <joint name="torso_joint1" type="revolute">
             <parent link="base_link"/><child link="torso_link1"/>
-            <origin xyz="-0.032845 0 0.301" rpy="-1.5708 0 0"/><axis xyz="0 0 1"/>
-            <limit lower="-1.1345" upper="1.8326" effort="100" velocity="2.5"/>
+            <origin xyz="-0.079032 0 0.34865" rpy="0 0 0"/><axis xyz="0 1 0"/>
+            <limit lower="-1.27354671" upper="1.81254671" effort="100" velocity="2.5"/>
         </joint>
         <link name="torso_link1">
             <inertial>
-                <origin xyz="0.00065636 -0.23142 0.0032247" rpy="0 0 0"/>
-                <mass value="10"/>
-                <inertia ixx="0.30931" ixy="0.00017473" ixz="0.00000779" iyy="0.0081222" iyz="-0.00013763" izz="0.30736"/>
+                <origin xyz="0.00065636 0.0032244 0.23142" rpy="0 0 0"/>
+                <mass value="5.72"/>
+                <inertia ixx="0.10931" ixy="0.00000779" ixz="-0.00017473" iyy="0.10736" iyz="0.00013778" izz="0.0081222"/>
             </inertial>
             <visual>
@@ -33,12 +35,12 @@
         <joint name="torso_joint2" type="revolute">
             <parent link="torso_link1"/><child link="torso_link2"/>
-            <origin xyz="0 -0.4 0" rpy="0 0 0"/><axis xyz="0 0 1"/>
-            <limit lower="-2.7925" upper="2.5307" effort="100" velocity="2.5"/>
+            <origin xyz="0 0 0.35" rpy="0 0 0"/><axis xyz="0 1 0"/>
+            <limit lower="-2.67034671" upper="2.68254671" effort="100" velocity="2.5"/>
         </joint>
         <link name="torso_link2">
             <inertial>
-                <origin xyz="0.0052517 -0.15711 0.014411" rpy="0 0 0"/>
-                <mass value="3.4"/>
-                <inertia ixx="0.026081" ixy="-0.00024541" ixz="-0.00000033" iyy="0.0018515" iyz="-0.00000038" izz="0.027574"/>
+                <origin xyz="0.0052517 0.014411 0.15711" rpy="0 0 0"/>
+                <mass value="3.5"/>
+                <inertia ixx="0.026081" ixy="-0.00000033" ixz="0.00024541" iyy="0.027574" iyz="0.00000042" izz="0.0018515"/>
             </inertial>
             <visual>
@@ -49,12 +51,12 @@
         <joint name="torso_joint3" type="revolute">
             <parent link="torso_link2"/><child link="torso_link3"/>
-            <origin xyz="0 -0.3 0" rpy="0 0 0"/><axis xyz="0 0 -1"/>
-            <limit lower="-2.0944" upper="1.8326" effort="100" velocity="2.5"/>
+            <origin xyz="0 0 0.35" rpy="0 0 0"/><axis xyz="0 -1 0"/>
+            <limit lower="-1.70954671" upper="1.53584671" effort="100" velocity="2.5"/>
         </joint>
         <link name="torso_link3">
             <inertial>
-                <origin xyz="-0.00000008 -0.031308 -0.00018966" rpy="0 0 0"/>
-                <mass value="5.5"/>
-                <inertia ixx="0.0035869" ixy="0" ixz="0" iyy="0.0036236" iyz="-0.00010486" izz="0.0043819"/>
+                <origin xyz="-0.00000098 -0.0055146 0.020182" rpy="0 0 0"/>
+                <mass value="3.4"/>
+                <inertia ixx="0.0016099" ixy="0.00000036" ixz="0.00000025" iyy="0.0023011" iyz="0.00001367" izz="0.0017027"/>
             </inertial>
             <visual>
@@ -65,12 +67,12 @@
         <joint name="torso_joint4" type="revolute">
             <parent link="torso_link3"/><child link="torso_link4"/>
-            <origin xyz="0 -0.12474 0" rpy="1.5708 0 0"/><axis xyz="0 0 1"/>
-            <limit lower="-3.0543" upper="3.0543" effort="100" velocity="2.5"/>
+            <origin xyz="0 -0.0010063 0.075322" rpy="0 0 0"/><axis xyz="0 0 1"/>
+            <limit lower="-3.01939342" upper="3.01939342" effort="100" velocity="2.5"/>
         </joint>
         <link name="torso_link4">
             <inertial>
-                <origin xyz="-0.0025153 0.00000031 0.35873" rpy="0 0 0"/>
-                <mass value="16.778"/>
-                <inertia ixx="0.015187" ixy="0.00000007" ixz="0.00054617" iyy="0.013478" iyz="-0.0000002" izz="0.017316"/>
+                <origin xyz="0.0049601 -0.0000125 0.21237" rpy="0 0 0"/>
+                <mass value="5"/>
+                <inertia ixx="0.026836" ixy="0.00001305" ixz="-0.00014074" iyy="0.013023" iyz="0.00000047" izz="0.021541"/>
             </inertial>
             <visual>
@@ -79,14 +81,24 @@
             </visual>
         </link>
+        <joint name="left_arm_base_joint" type="fixed">
+            <parent link="torso_link4"/><child link="left_arm_base_link"/>
+            <origin xyz="-0.00047402 0.097235 0.32738" rpy="0 0 -0.00070441"/>
+        </joint>
+        <link name="left_arm_base_link"/>
+        <joint name="right_arm_base_joint" type="fixed">
+            <parent link="torso_link4"/><child link="right_arm_base_link"/>
+            <origin xyz="-0.00061101 -0.097235 0.32738" rpy="0 0 -0.00070441"/>
+        </joint>
+        <link name="right_arm_base_link"/>
         <joint name="left_arm_joint1" type="revolute">
-            <parent link="torso_link4"/><child link="left_arm_link1"/>
-            <origin xyz="-0.00033786 0.13608 0.27773" rpy="-1.5708 0 0"/><axis xyz="0 0 1"/>
-            <limit lower="-2.8798" upper="2.8798" effort="40" velocity="20.944"/>
+            <parent link="left_arm_base_link"/><child link="left_arm_link1"/>
+            <origin xyz="0 0.0735 0" rpy="0 0 0"/><axis xyz="0 1 0"/>
+            <limit lower="-4.41569341" upper="1.27409342" effort="55" velocity="7.1209"/>
         </joint>
         <link name="left_arm_link1">
             <inertial>
-                <origin xyz="0.0020734 0.00846 0.19171" rpy="0 0 0"/>
-                <mass value="1.319"/>
-                <inertia ixx="0.00058101" ixy="0.00000001" ixz="0.00000003" iyy="0.00070857" iyz="0.00000086" izz="0.00044583"/>
+                <origin xyz="0.00042258 0.074131 0.00007916" rpy="0 0 0"/>
+                <mass value="1.135"/>
+                <inertia ixx="0.00061603" ixy="-0.00000116" ixz="-0.0000007" iyy="0.00030259" iyz="-0.00000063" izz="0.00047136"/>
             </inertial>
             <visual>
@@ -97,12 +109,12 @@
         <joint name="left_arm_joint2" type="revolute">
             <parent link="left_arm_link1"/><child link="left_arm_link2"/>
-            <origin xyz="0 0 0.11185" rpy="-1.5708 0 0"/><axis xyz="0 0 1"/>
-            <limit lower="0" upper="3.2289" effort="40" velocity="20.944"/>
+            <origin xyz="0.025012 0.081265 0" rpy="0 0 0"/><axis xyz="1 0 0"/>
+            <limit lower="-0.13959341" upper="3.10669342" effort="55" velocity="7.1209"/>
         </joint>
         <link name="left_arm_link2">
             <inertial>
-                <origin xyz="-0.23622 -0.016352 0.00013272" rpy="0 0 0"/>
-                <mass value="1.3"/>
-                <inertia ixx="0.00060638" ixy="0.00004182" ixz="-0.00014956" iyy="0.0075936" iyz="0.00000809" izz="0.0075712"/>
+                <origin xyz="-0.026826 -0.0040392 -0.031835" rpy="0 0 0"/>
+                <mass value="0.92"/>
+                <inertia ixx="0.00037378" ixy="-0.00000076" ixz="0.0000029" iyy="0.00033872" iyz="0.00001217" izz="0.00032361"/>
             </inertial>
             <visual>
@@ -113,12 +125,12 @@
         <joint name="left_arm_joint3" type="revolute">
             <parent link="left_arm_link2"/><child link="left_arm_link3"/>
-            <origin xyz="-0.34928 -0.019999 0" rpy="0 0 0"/><axis xyz="0 0 1"/>
-            <limit lower="-3.3161" upper="0" effort="27" velocity="7.5398"/>
+            <origin xyz="-0.025012 0 -0.1155" rpy="0 0 0"/><axis xyz="0 0 1"/>
+            <limit lower="-2.32128941" upper="2.32128941" effort="25" velocity="8.3776"/>
         </joint>
         <link name="left_arm_link3">
             <inertial>
-                <origin xyz="0.045114 -0.054616 0.00045585" rpy="0 0 0"/>
-                <mass value="0.818"/>
-                <inertia ixx="0.00060107" ixy="0.00022467" ixz="0.00000712" iyy="0.0013959" iyz="-0.00000975" izz="0.0015027"/>
+                <origin xyz="0.0053849 -0.00086892 -0.1126" rpy="0 0 0"/>
+                <mass value="1.245"/>
+                <inertia ixx="0.00072339" ixy="-0.00000335" ixz="-0.00012824" iyy="0.00073856" iyz="-0.00000836" izz="0.00037352"/>
             </inertial>
             <visual>
@@ -129,12 +141,12 @@
         <joint name="left_arm_joint4" type="revolute">
             <parent link="left_arm_link3"/><child link="left_arm_link4"/>
-            <origin xyz="0.02735 -0.069767 0" rpy="-3.1416 1.5708 3.1416"/><axis xyz="0 0 1"/>
-            <limit lower="-2.8798" upper="2.8798" effort="7" velocity="25.133"/>
+            <origin xyz="0 0.035065 -0.1945" rpy="0 0 0"/><axis xyz="0 1 0"/>
+            <limit lower="-2.05949341" upper="0.31419341" effort="25" velocity="8.3776"/>
         </joint>
         <link name="left_arm_link4">
             <inertial>
-                <origin xyz="0.00000082 -0.0023773 0.24285" rpy="0 0 0"/>
-                <mass value="0.816"/>
-                <inertia ixx="0.00009704" ixy="-0.00000001" ixz="0" iyy="0.00010174" iyz="0.00000083" izz="0.0000845"/>
+                <origin xyz="-0.0011018 -0.036243 -0.042164" rpy="0 0 0"/>
+                <mass value="0.827"/>
+                <inertia ixx="0.00013884" ixy="0.00000008" ixz="0.00000359" iyy="0.00019751" iyz="0.00000142" izz="0.00010229"/>
             </inertial>
             <visual>
@@ -145,12 +157,12 @@
         <joint name="left_arm_joint5" type="revolute">
             <parent link="left_arm_link4"/><child link="left_arm_link5"/>
-            <origin xyz="0 -0.0025 0.2463" rpy="1.5708 -1.5703 0.0077846"/><axis xyz="0 0 1"/>
-            <limit lower="-1.6581" upper="1.6581" effort="7" velocity="25.133"/>
+            <origin xyz="0 -0.035065 -0.095" rpy="0 0 0"/><axis xyz="0 0 1"/>
+            <limit lower="-2.32128941" upper="2.32128941" effort="18" velocity="10.472"/>
         </joint>
         <link name="left_arm_link5">
             <inertial>
-                <origin xyz="0.054309 0.00003483 0.0011809" rpy="0 0 0"/>
-                <mass value="0.801"/>
-                <inertia ixx="0.000084" ixy="0.00000004" ixz="0.00001623" iyy="0.00011332" iyz="-0.00000009" izz="0.0000985"/>
+                <origin xyz="0.00000038 -0.0028035 -0.062981" rpy="0 0 0"/>
+                <mass value="0.939"/>
+                <inertia ixx="0.00070496" ixy="0.00000001" ixz="0" iyy="0.00067006" iyz="-0.00005195" izz="0.00032998"/>
             </inertial>
             <visual>
@@ -161,12 +173,12 @@
         <joint name="left_arm_joint6" type="revolute">
             <parent link="left_arm_link5"/><child link="left_arm_link6"/>
-            <origin xyz="0.16215 0.00006892 -0.0024999" rpy="-1.5708 -0.0077846 -1.5702"/><axis xyz="0 0 1"/>
-            <limit lower="-2.8798" upper="2.8798" effort="7" velocity="25.133"/>
+            <origin xyz="0 -0.028 -0.16305" rpy="0 0 0"/><axis xyz="0 1 0"/>
+            <limit lower="-1.01229141" upper="1.01229141" effort="18" velocity="10.472"/>
         </joint>
         <link name="left_arm_link6">
             <inertial>
-                <origin xyz="-0.00000015 0.00000007 -0.031107" rpy="0 0 0"/>
-                <mass value="0.465"/>
-                <inertia ixx="0.00016512" ixy="0.00000008" ixz="0" iyy="0.00009864" iyz="0" izz="0.00017588"/>
+                <origin xyz="0.0017919 0.027487 0.00025471" rpy="0 0 0"/>
+                <mass value="0.527"/>
+                <inertia ixx="0.00008544" ixy="-0.00000015" ixz="0.00000084" iyy="0.00008119" iyz="-0.00000002" izz="0.00008274"/>
             </inertial>
             <visual>
@@ -175,14 +187,30 @@
             </visual>
         </link>
+        <joint name="left_arm_joint7" type="revolute">
+            <parent link="left_arm_link6"/><child link="left_arm_link7"/>
+            <origin xyz="0.0295 0.028 0" rpy="0 0 0"/><axis xyz="1 0 0"/>
+            <limit lower="-1.53589342" upper="1.53589342" effort="18" velocity="10.472"/>
+        </joint>
+        <link name="left_arm_link7">
+            <inertial>
+                <origin xyz="-0.022945 0.00000084 -0.056525" rpy="0 0 0"/>
+                <mass value="0.185"/>
+                <inertia ixx="0.00004256" ixy="0" ixz="-0.00000694" iyy="0.00004552" iyz="0" izz="0.00004795"/>
+            </inertial>
+            <visual>
+                <origin xyz="0 0 0" rpy="0 0 0"/>
+                <geometry><mesh filename="package://unistackbot_description/mobile_manipulators/r1_pro/meshes/left_arm_link7.STL"/></geometry>
+            </visual>
+        </link>
         <joint name="right_arm_joint1" type="revolute">
-            <parent link="torso_link4"/><child link="right_arm_link1"/>
-            <origin xyz="-0.0003367 -0.13609 0.27773" rpy="1.5786 -0.00054698 0"/><axis xyz="0 0 1"/>
-            <limit lower="-2.8798" upper="2.8798" effort="40" velocity="20.944"/>
+            <parent link="right_arm_base_link"/><child link="right_arm_link1"/>
+            <origin xyz="0 -0.0735 0" rpy="0 0 0"/><axis xyz="0 1 0"/>
+            <limit lower="-4.41569341" upper="1.27409342" effort="55" velocity="7.1209"/>
         </joint>
         <link name="right_arm_link1">
             <inertial>
-                <origin xyz="0.0020139 0.0089421 0.19171" rpy="0 0 0"/>
-                <mass value="1.319"/>
-                <inertia ixx="0.00058101" ixy="-0.00000001" ixz="-0.00000003" iyy="0.00070857" iyz="0.00000086" izz="0.00044583"/>
+                <origin xyz="-0.00042261 -0.074132 0.00007836" rpy="0 0 0"/>
+                <mass value="1.135"/>
+                <inertia ixx="0.00061603" ixy="-0.00000116" ixz="0.0000007" iyy="0.00030259" iyz="0.00000062" izz="0.00047135"/>
             </inertial>
             <visual>
@@ -193,12 +221,12 @@
         <joint name="right_arm_joint2" type="revolute">
             <parent link="right_arm_link1"/><child link="right_arm_link2"/>
-            <origin xyz="0 0.00087053 0.11185" rpy="-1.5786 0 -0.00054696"/><axis xyz="0 0 1"/>
-            <limit lower="0" upper="3.2289" effort="40" velocity="20.944"/>
+            <origin xyz="0.023988 -0.081265 0" rpy="0 0 0"/><axis xyz="1 0 0"/>
+            <limit lower="-3.10669342" upper="0.13959341" effort="55" velocity="7.1209"/>
         </joint>
         <link name="right_arm_link2">
             <inertial>
-                <origin xyz="-0.23622 -0.016354 0.00013181" rpy="0 0 0"/>
-                <mass value="1.3"/>
-                <inertia ixx="0.00060639" ixy="-0.00041823" ixz="-0.00014959" iyy="0.0075936" iyz="-0.00000809" izz="0.0075712"/>
+                <origin xyz="-0.022361 0.0049527 -0.032732" rpy="0 0 0"/>
+                <mass value="0.92"/>
+                <inertia ixx="0.00038179" ixy="0.00000027" ixz="-0.00000364" iyy="0.00034188" iyz="-0.00000844" izz="0.00032895"/>
             </inertial>
             <visual>
@@ -209,12 +237,12 @@
         <joint name="right_arm_joint3" type="revolute">
             <parent link="right_arm_link2"/><child link="right_arm_link3"/>
-            <origin xyz="-0.34928 -0.020001 0" rpy="0 0 0"/><axis xyz="0 0 1"/>
-            <limit lower="-3.3161" upper="0" effort="27" velocity="7.5398"/>
+            <origin xyz="-0.023988 0 -0.1155" rpy="0 0 0"/><axis xyz="0 0 1"/>
+            <limit lower="-2.32128941" upper="2.32128941" effort="25" velocity="8.3776"/>
         </joint>
         <link name="right_arm_link3">
             <inertial>
-                <origin xyz="0.045115 -0.054616 0.00045605" rpy="0 0 0"/>
-                <mass value="0.818"/>
-                <inertia ixx="0.00060107" ixy="0.00022466" ixz="0.00000712" iyy="0.0013959" iyz="-0.00000975" izz="0.0015027"/>
+                <origin xyz="0.0053839 -0.00087109 -0.11261" rpy="0 0 0"/>
+                <mass value="1.245"/>
+                <inertia ixx="0.00072336" ixy="-0.00000336" ixz="-0.00012821" iyy="0.00073854" iyz="-0.00000837" izz="0.00037348"/>
             </inertial>
             <visual>
@@ -225,12 +253,12 @@
         <joint name="right_arm_joint4" type="revolute">
             <parent link="right_arm_link3"/><child link="right_arm_link4"/>
-            <origin xyz="0.02735 -0.069767 0" rpy="0 -1.5708 3.1416"/><axis xyz="0 0 1"/>
-            <limit lower="-2.8798" upper="2.8798" effort="7" velocity="25.133"/>
+            <origin xyz="0 0.035058 -0.1945" rpy="0 0 0"/><axis xyz="0 1 0"/>
+            <limit lower="-2.05949341" upper="0.31419341" effort="25" velocity="8.3776"/>
         </joint>
         <link name="right_arm_link4">
             <inertial>
-                <origin xyz="-0.00000082 0.0023773 0.24285" rpy="0 0 0"/>
-                <mass value="0.816"/>
-                <inertia ixx="0.00009704" ixy="-0.00000001" ixz="0" iyy="0.00010174" iyz="-0.00000083" izz="0.0000845"/>
+                <origin xyz="-0.00058877 -0.035687 -0.057422" rpy="0 0 0"/>
+                <mass value="0.827"/>
+                <inertia ixx="0.00016157" ixy="0.00000008" ixz="0.00000359" iyy="0.00022024" iyz="0.00000142" izz="0.00012683"/>
             </inertial>
             <visual>
@@ -241,12 +269,12 @@
         <joint name="right_arm_joint5" type="revolute">
             <parent link="right_arm_link4"/><child link="right_arm_link5"/>
-            <origin xyz="0 0.0025 0.2463" rpy="-1.5708 -1.5703 0.0077846"/><axis xyz="0 0 1"/>
-            <limit lower="-1.6581" upper="1.6581" effort="7" velocity="25.133"/>
+            <origin xyz="0 -0.035058 -0.095" rpy="0 0 0"/><axis xyz="0 0 1"/>
+            <limit lower="-2.32128941" upper="2.32128941" effort="18" velocity="10.472"/>
         </joint>
         <link name="right_arm_link5">
             <inertial>
-                <origin xyz="0.054309 -0.00002438 0.0011809" rpy="0 0 0"/>
-                <mass value="0.801"/>
-                <inertia ixx="0.000084" ixy="0.00000007" ixz="0.00001623" iyy="0.00011332" iyz="-0.00000011" izz="0.0000985"/>
+                <origin xyz="-0.00000023 0.0031762 -0.07334" rpy="0 0 0"/>
+                <mass value="0.63"/>
+                <inertia ixx="0.00069134" ixy="0.00000001" ixz="0" iyy="0.00065644" iyz="0.00005195" izz="0.00031157"/>
             </inertial>
             <visual>
@@ -257,16 +285,32 @@
         <joint name="right_arm_joint6" type="revolute">
             <parent link="right_arm_link5"/><child link="right_arm_link6"/>
-            <origin xyz="0.16215 -0.00010784 -0.0024999" rpy="1.5708 0 1.5703"/><axis xyz="0 0 1"/>
-            <limit lower="-2.8798" upper="2.8798" effort="7" velocity="25.133"/>
+            <origin xyz="0 0.028001 -0.16305" rpy="0 0 0"/><axis xyz="0 1 0"/>
+            <limit lower="-1.01229141" upper="1.01229141" effort="18" velocity="10.472"/>
         </joint>
         <link name="right_arm_link6">
             <inertial>
-                <origin xyz="-0.00000002 -0.00000006 -0.031107" rpy="0 0 0"/>
-                <mass value="0.465"/>
-                <inertia ixx="0.00016512" ixy="-0.00000044" ixz="0" iyy="0.00009864" iyz="0" izz="0.00017588"/>
+                <origin xyz="0.0017914 -0.027486 0.00025485" rpy="0 0 0"/>
+                <mass value="0.527"/>
+                <inertia ixx="0.00008544" ixy="0.00000015" ixz="0.00000084" iyy="0.00008119" iyz="0.00000002" izz="0.00008274"/>
             </inertial>
             <visual>
                 <origin xyz="0 0 0" rpy="0 0 0"/>
                 <geometry><mesh filename="package://unistackbot_description/mobile_manipulators/r1_pro/meshes/right_arm_link6.STL"/></geometry>
+            </visual>
+        </link>
+        <joint name="right_arm_joint7" type="revolute">
+            <parent link="right_arm_link6"/><child link="right_arm_link7"/>
+            <origin xyz="0.0295 -0.028001 0" rpy="0 0 0"/><axis xyz="1 0 0"/>
+            <limit lower="-1.53589342" upper="1.53589342" effort="18" velocity="10.472"/>
+        </joint>
+        <link name="right_arm_link7">
+            <inertial>
+                <origin xyz="-0.022945 0.00000023 -0.056523" rpy="0 0 0"/>
+                <mass value="0.185"/>
+                <inertia ixx="0.00007854" ixy="0" ixz="-0.00002871" iyy="0.00009467" iyz="0" izz="0.00006113"/>
+            </inertial>
+            <visual>
+                <origin xyz="0 0 0" rpy="0 0 0"/>
+                <geometry><mesh filename="package://unistackbot_description/mobile_manipulators/r1_pro/meshes/right_arm_link7.STL"/></geometry>
             </visual>
         </link>
