Commit message: 底盘域B阶段:N舵轮运动学+r1_pro三舵轮上gz

File: unistackbot_description/mobile_manipulators/r1_pro/urdf/r1_pro.ros2_control.xacro (robot description, xacro)
@@ -55,4 +55,26 @@
             <xacro:r1_joint name="torso_joint3" lo="-1.7095467075" hi="1.5358467075"/>
             <xacro:r1_joint name="torso_joint4" lo="-3.0193934150" hi="3.0193934150"/>
+            <!-- 轮系 6 (仅 gz/mujoco 链, 与 body 轮 link 同条件; steer=position 归
+                 BaseVelocityController, yaml joints 显式列表不含它 = JS 不认领) -->
+            <xacro:if value="${use_gazebo in ['ign', 'mujoco']}">
+                <xacro:macro name="r1_wheel_joint" params="idx">
+                    <joint name="steer_motor_joint${idx}">
+                        <command_interface name="position"/>
+                        <state_interface name="position"/>
+                        <state_interface name="velocity"/>
+                        <param name="min">-3.14</param>
+                        <param name="max">3.14</param>
+                        <param name="max_velocity">6.0</param>
+                    </joint>
+                    <joint name="wheel_motor_joint${idx}">
+                        <command_interface name="velocity"/>
+                        <state_interface name="position"/>
+                        <state_interface name="velocity"/>
+                    </joint>
+                </xacro:macro>
+                <xacro:r1_wheel_joint idx="1"/>
+                <xacro:r1_wheel_joint idx="2"/>
+                <xacro:r1_wheel_joint idx="3"/>
+            </xacro:if>
         </ros2_control>
         <!-- Gazebo 侧系统插件 (ign 三件之二; 三 = 易冻关节 initial_value, 指纹后按需) -->

File: unistackbot_description/mobile_manipulators/r1_pro/urdf/r1_pro.urdf.xacro (robot description, xacro)
@@ -2,6 +2,8 @@
 <robot xmlns:xacro="http://www.ros.org/wiki/xacro" name="r1_pro">
     <!-- r1_pro 顶层入口 (Galaxea R1 Pro, 2026-10-14 接入)
-         五参数同 piper 范本; body 宏只含控制域 16 关节 (腰4+双臂12, 四件式分割),
-         轮域分离式接入暂不声明 (底盘生态件后续按需)。 -->
+         五参数同 piper 范本; body 宏 = 控制域 18 关节 (腰4+双臂14, 四件式分割)。
+         轮域 (2026-10-15 底盘域 B2): 三舵轮模块仅 gz/mujoco 链声明 (mock 无世界
+         语义不声明, 用户裁决); 该两链同时去掉 world 固定关节 —— 底盘要动, 基座
+         必须浮动 (gz spawn 自由体, 物理由三轮支撑)。 -->
     <xacro:arg name="use_gripper" default="true"/>
     <xacro:arg name="use_ros2_control" default="false"/>
@@ -9,12 +11,20 @@
     <xacro:arg name="use_gazebo" default="false"/>
     <xacro:arg name="headless" default="true"/>
+    <xacro:property name="ug" value="$(arg use_gazebo)"/>
+    <xacro:property name="mobile_chain" value="${ug in ['ign', 'mujoco']}"/>
     <xacro:include filename="$(find unistackbot_description)/mobile_manipulators/r1_pro/urdf/r1_pro_macro.xacro"/>
     <xacro:include filename="$(find unistackbot_description)/mobile_manipulators/r1_pro/urdf/r1_pro.ros2_control.xacro"/>
+    <xacro:include filename="$(find unistackbot_description)/mobile_manipulators/r1_pro/urdf/r1_pro_wheels.xacro"/>
     <xacro:r1_pro_body/>
+    <xacro:if value="${mobile_chain}">
+        <xacro:r1_pro_wheels/>
+    </xacro:if>
     <xacro:if value="$(arg use_world)">
-        <link name="world"/>
-        <joint name="r1_pro_world" type="fixed">
-            <parent link="world"/><child link="base_link"/>
-        </joint>
+        <xacro:if value="${not mobile_chain}">
+            <link name="world"/>
+            <joint name="r1_pro_world" type="fixed">
+                <parent link="world"/><child link="base_link"/>
+            </joint>
+        </xacro:if>
     </xacro:if>
     <xacro:if value="$(arg use_ros2_control)">
